Commit message: Still has some ROS2 and macos compatibility bugs

File: omni_ws/src/omni_description/urdf/gazebo.xacro (robot description, xacro)
@@ -2,40 +2,43 @@
 <robot xmlns:xacro="http://www.ros.org/wiki/xacro">
   <!-- ============================================================
-       Gazebo (Classic 11) material + sensor + plugin definitions.
-       Paired with ROS 2 Humble via gazebo_ros_pkgs.
+       Gazebo Sim (Fortress / gz-sim6) extensions.
+       Paired with ROS 2 Humble via ros_gz.
+       Motion:   VelocityControl (holonomic — body-frame vx, vy, wz)
+       Odometry: OdometryPublisher (odom -> base_footprint)
+       Sensors:  gpu_lidar, imu, camera
+       Topics are bridged to ROS 2 by ros_gz_bridge (see omni_gazebo).
        ============================================================ -->
-  <!-- Visual materials in Gazebo -->
+  <!-- Visual materials in Gazebo Sim -->
   <gazebo reference="base_link"><material>Gazebo/Grey</material></gazebo>
-  <gazebo reference="fl_wheel_link"><material>Gazebo/Black</material></gazebo>
-  <gazebo reference="fr_wheel_link"><material>Gazebo/Black</material></gazebo>
-  <gazebo reference="rl_wheel_link"><material>Gazebo/Black</material></gazebo>
-  <gazebo reference="rr_wheel_link"><material>Gazebo/Black</material></gazebo>
-  <gazebo reference="lidar_link"><material>Gazebo/Orange</material></gazebo>
-  <gazebo reference="camera_link"><material>Gazebo/Black</material></gazebo>
+  <gazebo reference="lidar_link"><visual><material><ambient>0.9 0.45 0.1 1</ambient><diffuse>0.9 0.45 0.1 1</diffuse></material></visual></gazebo>
   <!-- ============================================================
-       Holonomic (mecanum) drive.
-       gazebo_ros_planar_move consumes geometry_msgs/Twist on /cmd_vel
-       (linear.x, linear.y AND angular.z) and publishes odom -> base.
-       This reproduces true omni-directional motion without modelling
-       each roller, which is ideal for an MVP.
+       Holonomic (mecanum) motion.
+       VelocityControl applies the commanded body-frame twist
+       (linear.x, linear.y, angular.z) directly to the model — the
+       gz-sim analogue of Classic's planar_move, ideal for an MVP.
+       Subscribes to gz topic /cmd_vel (bridged from ROS /cmd_vel).
        ============================================================ -->
   <gazebo>
-    <plugin name="planar_move_controller" filename="libgazebo_ros_planar_move.so">
-      <ros>
-        <namespace>/</namespace>
-        <remapping>cmd_vel:=cmd_vel</remapping>
-        <remapping>odom:=odom</remapping>
-      </ros>
-      <update_rate>50</update_rate>
-      <publish_rate>50</publish_rate>
-      <odometry_frame>odom</odometry_frame>
-      <robot_base_frame>base_footprint</robot_base_frame>
-      <covariance_x>0.0001</covariance_x>
-      <covariance_y>0.0001</covariance_y>
-      <covariance_yaw>0.01</covariance_yaw>
+    <plugin filename="ignition-gazebo-velocity-control-system"
+            name="ignition::gazebo::systems::VelocityControl">
+      <topic>cmd_vel</topic>
     </plugin>
   </gazebo>
   <!-- ============================================================
-       IMU sensor (GY-9250 stand-in)
+       Wheel odometry: publishes gz.msgs.Odometry on
+       /model/omni_bot/odometry and the odom->base_footprint TF on
+       /model/omni_bot/tf (both bridged to ROS).
+       ============================================================ -->
+  <gazebo>
+    <plugin filename="ignition-gazebo-odometry-publisher-system"
+            name="ignition::gazebo::systems::OdometryPublisher">
+      <odom_frame>odom</odom_frame>
+      <robot_base_frame>base_footprint</robot_base_frame>
+      <odom_publish_frequency>50</odom_publish_frequency>
+      <dimensions>2</dimensions>
+    </plugin>
+  </gazebo>
+  <!-- ============================================================
+       IMU sensor (GY-9250 stand-in). Needs the Imu system in the world.
        ============================================================ -->
   <gazebo reference="imu_link">
@@ -43,13 +46,5 @@
       <always_on>true</always_on>
       <update_rate>100</update_rate>
-      <visualize>false</visualize>
-      <plugin name="imu_plugin" filename="libgazebo_ros_imu_sensor.so">
-        <ros>
-          <namespace>/</namespace>
-          <remapping>~/out:=imu/data</remapping>
-        </ros>
-        <initial_orientation_as_reference>false</initial_orientation_as_reference>
-        <frame_name>imu_link</frame_name>
-      </plugin>
+      <topic>imu/data</topic>
       <imu>
         <angular_velocity>
@@ -67,5 +62,6 @@
   </gazebo>
   <!-- ============================================================
-       Pi Camera 3 (RGB)
+       Pi Camera 3 (RGB). Needs the Sensors (rendering) system.
+       Publishes /pi_camera/image and /pi_camera/camera_info.
        ============================================================ -->
   <gazebo reference="camera_link">
@@ -73,26 +69,23 @@
       <always_on>true</always_on>
       <update_rate>30</update_rate>
-      <visualize>true</visualize>
-      <camera name="pi_cam">
+      <topic>pi_camera</topic>
+      <camera>
         <horizontal_fov>1.204</horizontal_fov>
         <image><width>640</width><height>480</height><format>R8G8B8</format></image>
         <clip><near>0.05</near><far>15.0</far></clip>
       </camera>
-      <plugin name="camera_plugin" filename="libgazebo_ros_camera.so">
-        <ros><namespace>/</namespace></ros>
-        <camera_name>pi_camera</camera_name>
-        <frame_name>camera_optical_link</frame_name>
-      </plugin>
     </sensor>
   </gazebo>
   <!-- ============================================================
-       2D Lidar (simulation only — provides /scan for Nav2 + AMCL)
+       2D Lidar (gpu_lidar) — SIMULATION ONLY, provides /scan for
+       Nav2 + AMCL. Needs the Sensors (rendering) system in the world.
        ============================================================ -->
   <gazebo reference="lidar_link">
-    <sensor name="lidar" type="ray">
+    <sensor name="lidar" type="gpu_lidar">
       <always_on>true</always_on>
       <update_rate>10</update_rate>
-      <visualize>true</visualize>
-      <ray>
+      <topic>scan</topic>
+      <gz_frame_id>lidar_link</gz_frame_id>
+      <lidar>
         <scan>
           <horizontal>
@@ -102,4 +95,9 @@
             <max_angle>3.14159</max_angle>
           </horizontal>
+          <vertical>
+            <samples>1</samples>
+            <min_angle>0</min_angle>
+            <max_angle>0</max_angle>
+          </vertical>
         </scan>
         <range>
@@ -109,13 +107,5 @@
         </range>
         <noise><type>gaussian</type><mean>0.0</mean><stddev>0.01</stddev></noise>
-      </ray>
-      <plugin name="lidar_plugin" filename="libgazebo_ros_ray_sensor.so">
-        <ros>
-          <namespace>/</namespace>
-          <remapping>~/out:=scan</remapping>
-        </ros>
-        <output_type>sensor_msgs/LaserScan</output_type>
-        <frame_name>lidar_link</frame_name>
-      </plugin>
+      </lidar>
     </sensor>
   </gazebo>
